File: Hardware/AnkleDynamometer/AnkleDynamometer.kicad_pcb (KiCad board)
At the start: 2 copper layers, 68 x 45 mm, 32 parts, among them J1 Conn_01x04, J2 Conn_01x08, J3 Barrel_Jack, J4 Conn_01x02, J5 Conn_01x02, SW1 SW_SPDT, U1 INA129, U2 LT3080xMS8E, U3 ADS1220xPW, U5 AMS1117-2.5

Commit message: PCB layout 2
Parts:
- added H1: MountingHole, MountingHole:MountingHole_2.2mm_M2_Pad_Via, F.Cu at (73.7, 106.7)
- added H2: MountingHole, MountingHole:MountingHole_2.2mm_M2_Pad_Via, F.Cu at (136.3, 106.7)
- added H3: MountingHole, MountingHole:MountingHole_2.2mm_M2_Pad_Via, F.Cu at (73.7, 146.3)
- added H4: MountingHole, MountingHole:MountingHole_2.2mm_M2_Pad_Via, F.Cu at (136.3, 146.3)
- C1, C10, C11: value 1 micro -> 1u; footprint Capacitor_SMD:C_0603_1608Metric -> Capacitor_SMD:C_0805_2012Metric
- C2: value 2.2 micro -> 2.2u; footprint Capacitor_SMD:C_0805_2012Metric -> Capacitor_SMD:C_1206_3216Metric
- C3, C4, C5, C7: value 0.1 micro -> 100n
- C6: value 10 nano -> 10n
- C8: value 22 micro -> 22u
- C9: value 10 micro -> 10u
- R1, R10, R2: footprint Resistor_SMD:R_0805_2012Metric_Pad1.20x1.40mm_HandSolder -> Resistor_SMD:R_0603_1608Metric_Pad0.98x0.95mm_HandSolder
- R8, R9: value 5k -> 5.1k; footprint Resistor_SMD:R_0805_2012Metric_Pad1.20x1.40mm_HandSolder -> Resistor_SMD:R_0603_1608Metric_Pad0.98x0.95mm_HandSolder
- moved C10 0.46 mm to (75.9, 121.2)
- moved J3 0.40 mm to (128.8, 118.3)
- moved C1 0.32 mm to (108.3, 105.8)
- moved C2 0.25 mm to (108.5, 109.9)
Routing:
- net GND: track 81.8 -> 83.3 mm
Other:
- board size 68 x 45 mm -> 69 x 46 mm
- board text added: "+ -"
- board text added: "V1 | May 2026 | K. Smart"
- board text removed: "V1 | May 2026 | Kendra Smart"
