File: Hardware/AnkleDynamometer/AnkleDynamometer.kicad_pcb (KiCad board)
At the start: 2 copper layers, 69 x 46 mm, 36 parts, among them J1 Conn_01x04, J2 Conn_01x08, J3 Barrel_Jack, J4 Conn_01x02, J5 Conn_01x02, SW1 SW_SPDT, U1 INA129, U2 LT3080xMS8E, U3 ADS1220xPW, U5 AMS1117-2.5

Commit message: Reorganizing
Parts:
- added C12: 22u, Capacitor_Tantalum_SMD:CP_EIA-3216-18_Kemet-A, F.Cu at (90.8, 117.6)
- added C13: 10u, Capacitor_Tantalum_SMD:CP_EIA-3216-18_Kemet-A, F.Cu at (86.1, 116.3)
- added U4: AMS1117-5.0, Package_TO_SOT_SMD:SOT-223-3_TabPin2, F.Cu at (88.4, 123.2)
- moved R8 7.58 mm to (82.2, 122.1)
- moved R9 7.56 mm to (82.2, 125.5)
- moved U5 7.00 mm to (82.2, 143.7), turned to -90 degrees
- moved C9 6.97 mm to (77.4, 139.2), turned to 90 degrees
- moved C8 2.80 mm to (84.1, 138.2), turned to 0 degrees
- moved C10 2.14 mm to (73.8, 121.0)
- moved C3 2.10 mm to (75.5, 130.1)
- moved U3 2.10 mm to (81.0, 131.1)
- moved C7 2.05 mm to (78.9, 127.6)
- moved R1 2.00 mm to (83.6, 114.6)
- moved U1 1.99 mm to (81.1, 110.6)
- moved C4 1.91 mm to (75.5, 131.9)
- moved R10 1.68 mm to (76.0, 121.0)
- moved C6 1.28 mm to (77.8, 123.5)
- moved C5 1.10 mm to (78.6, 120.8)
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Connections:
- C7 pad 2: +5V -> Net-(U3-REFP0)
- R8 pad 2: +5V -> Net-(U3-REFP0)
- R9 pad 1: +5V -> Net-(U3-REFP0)
- U3 pad 9: +5V -> Net-(U3-REFP0)
Routing:
- net /2.5V: track 11.1 -> 45.6 mm
- net GND: track 83.3 -> 50.1 mm, vias 17 -> 21
- net +10V: track 50.6 -> 62.0 mm
- net Net-(U3-REFP0): track 0.00 -> 8.15 mm
- net Net-(U3-AIN1): track 7.19 -> 10.2 mm
- net Net-(U3-DIN): track 10.2 -> 12.4 mm
- net Net-(U3-~{CS}): track 4.86 -> 7.01 mm
- net Net-(U3-SCLK): track 4.51 -> 6.66 mm
- net Net-(J1-Pin_4): track 8.35 -> 10.4 mm
- net Net-(U3-DOUT/~{DRDY}): track 13.4 -> 15.2 mm
- net Net-(A1-+5V): track 129.9 -> 131.5 mm
- net Net-(J1-Pin_1): track 4.62 -> 6.04 mm
- net Net-(U3-~{DRDY}): track 15.5 -> 16.9 mm
- net +5V: track 48.8 -> 47.5 mm
- removed copper zone on F.Cu, net +10V
- removed copper zone on F.Cu, net /2.5V

Commit message: PCB Updates
Updating the PCB design based on testing of the previous design. Also re-exported and tested the production files so it is ready to upload to JLCPCB
Other:
- board text added: "- +"
Changed lines of the file:
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@@
 		(tags "capacitor tantalum")
 		(property "Reference" "C12"
-			(at -1.9012 -1.778 0)
+			(at 2.9248 1.3208 0)
 			(layer "F.SilkS")
 			(effects
@@
 		)
 	)
+	(gr_text "-\n\n+"
+		(at 87.122 118.0084 0)
+		(layer "F.SilkS")
+		(effects
+			(font
+				(size 0.8128 0.8128)
+				(thickness 0.1524)
+				(bold yes)
+			)
+			(justify left bottom)
+		)
+	)
 	(gr_text "+\n\n-"
 		(at 85.6996 137.16 90)
@@
 				(thickness 0.1524)
 				(bold yes)
+			)
+			(justify left bottom)
+		)
+	)
+	(gr_text "+  -"
+		(at 89.0016 116.4844 0)
+		(layer "F.SilkS")
+		(effects
+			(font
+				(size 0.8128 0.8128)
+				(thickness 0.1524)
+				(bold yes)
