File: Hardware/AnkleDynamometer/AnkleDynamometer.kicad_sch (KiCad schematic)
At the start: 36 parts, among them J1 Conn_01x04, J2 Conn_01x08, J3 Barrel_Jack, J4 Conn_01x02, J5 Conn_01x02, SW1 SW_SPDT, U1 INA129, U2 LT3080xMS8E, U3 ADS1220xPW, U5 AMS1117-2.5

Commit message: Reorganizing
Parts:
- added C12: 22u, Capacitor_Tantalum_SMD:CP_EIA-3216-18_Kemet-A, symbol Device:C_Polarized
- added C13: 10u, Capacitor_Tantalum_SMD:CP_EIA-3216-18_Kemet-A, symbol Device:C_Polarized
- added U4: AMS1117-5.0, Package_TO_SOT_SMD:SOT-223-3_TabPin2, symbol Regulator_Linear:AMS1117-5.0
Connections:
- net +10V: now also C13.1, U4.3 (VI)
- net +5V: now also C12.1, U4.2 (VO); no longer C7.2, R8.2, R9.1, U3.9 (REFP0)
- net GND: now also C12.2, C13.2, U4.1 (GND)
- new net: C7.2, R8.2, R9.1, U3.9 (REFP0)
Other:
- moved on the sheet: C1, C11, C2, H1, H2, H3, H4, J3, R2, R8, R9, SW1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
